File: PCB/PiFencePCB.kicad_sch (KiCad schematic)
At the start: 13 parts, among them J1 Barrel_Jack_MountingPin, J2 USB_Power_Breakout, J3 USB_Power_Breakout, J4 USB_Power_Breakout, J5 USB_Power_Breakout, J6 USB_Power_Breakout, J7 Conn_01x10_Socket, K1 Relay_SPDT, K2 Relay_SPDT, K3 Relay_SPDT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

Commit message: Added a PCB readme. Some small changes to the schematic
Parts:
- removed J7: Conn_01x10_Socket, Connector_PinSocket_2.54mm:PinSocket_2x05_P2.54mm_Vertical, symbol Connector:Conn_01x10_Socket
- added U2: ENC28J60x-SP, Package_DIP:DIP-28_W7.62mm, symbol Interface_Ethernet:ENC28J60x-SP
Changed lines of the file:
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@@
     (rev "0.1")
   )
-  (junction (at 104.14 127) (diameter 0) (color 0 0 0 0)
-  )
   (junction (at 218.44 125.73) (diameter 0) (color 0 0 0 0)
   )
@@
   (junction (at 73.66 54.61) (diameter 0) (color 0 0 0 0)
   )
-  (junction (at 104.14 156.21) (diameter 0) (color 0 0 0 0)
-  )
   (junction (at 201.93 87.63) (diameter 0) (color 0 0 0 0)
   )
@@
     (stroke (width 0) (type default))
   )
+  (wire (pts (xy 64.77 54.61) (xy 71.12 54.61))
+    (stroke (width 0) (type default))
+  )
   (wire (pts (xy 127 138.43) (xy 138.43 138.43))
     (stroke (width 0) (type default))
   )
-  (wire (pts (xy 97.79 111.76) (xy 104.14 111.76))
-    (stroke (width 0) (type default))
-  )
   (wire (pts (xy 71.12 48.26) (xy 71.12 54.61))
     (stroke (width 0) (type default))
   )
-  (wire (pts (xy 97.79 124.46) (xy 127 124.46))
-    (stroke (width 0) (type default))
-  )
   (wire (pts (xy 137.16 118.11) (xy 137.16 90.17))
     (stroke (width 0) (type default))
@@
     (stroke (width 0) (type default))
   )
-  (wire (pts (xy 49.53 54.61) (xy 71.12 54.61))
-    (stroke (width 0) (type default))
-  )
   (wire (pts (xy 114.3 77.47) (xy 114.3 91.44))
     (stroke (width 0) (type default))
@@
     (stroke (width 0) (type default))
   )
-  (wire (pts (xy 97.79 119.38) (xy 125.73 119.38))
-    (stroke (width 0) (type default))
-  )
   (wire (pts (xy 210.82 101.6) (xy 210.82 130.81))
     (stroke (width 0) (type default))
@@
     (stroke (width 0) (type default))
   )
-  (wire (pts (xy 104.14 111.76) (xy 104.14 127))
-    (stroke (width 0) (type default))
-  )
-  (wire (pts (xy 127 124.46) (xy 127 138.43))
-    (stroke (width 0) (type default))
-  )
   (wire (pts (xy 73.66 77.47) (xy 73.66 90.17))
     (stroke (width 0) (type default))
@@
     (stroke (width 0) (type default))
   )
-  (wire (pts (xy 97.79 114.3) (xy 124.46 114.3))
-    (stroke (width 0) (type default))
-  )
   (wire (pts (xy 231.14 54.61) (xy 232.41 54.61))
     (stroke (width 0) (type default))
@@
     (stroke (width 0) (type default))
   )
-  (wire (pts (xy 156.21 105.41) (xy 156.21 99.06))
-    (stroke (width 0) (type default))
-  )
   (wire (pts (xy 73.66 54.61) (xy 111.76 54.61))
     (stroke (width 0) (type default))
@@
     (stroke (width 0) (type default))
   )
-  (wire (pts (xy 104.14 127) (xy 104.14 156.21))
-    (stroke (width 0) (type default))
-  )
   (wire (pts (xy 127 55.88) (xy 127 48.26))
     (stroke (width 0) (type default))
@@
     (stroke (width 0) (type default))
   )
-  (wire (pts (xy 123.19 106.68) (xy 97.79 106.68))
-    (stroke (width 0) (type default))
-  )
-  (wire (pts (xy 124.46 114.3) (xy 124.46 146.05))
-    (stroke (width 0) (type default))
-  )
   (wire (pts (xy 138.43 120.65) (xy 135.89 120.65))
     (stroke (width 0) (type default))
@@
     (stroke (width 0) (type default))
   )
-  (wire (pts (xy 128.27 116.84) (xy 128.27 135.89))
-    (stroke (width 0) (type default))
-  )
   (wire (pts (xy 114.3 54.61) (xy 114.3 62.23))
     (stroke (width 0) (type default))
@@
     (stroke (width 0) (type default))
   )
-  (wire (pts (xy 49.53 54.61) (xy 49.53 156.21))
-    (stroke (width 0) (type default))
-  )
   (wire (pts (xy 111.76 48.26) (xy 111.76 54.61))
     (stroke (width 0) (type default))
@@
     (stroke (width 0) (type default))
   )
+  (wire (pts (xy 64.77 54.61) (xy 64.77 156.21))
+    (stroke (width 0) (type default))
+  )
   (wire (pts (xy 191.77 54.61) (xy 231.14 54.61))
     (stroke (width 0) (type default))
@@
     (stroke (width 0) (type default))
   )
-  (wire (pts (xy 156.21 99.06) (xy 123.19 99.06))
-    (stroke (width 0) (type default))
-  )
   (wire (pts (xy 151.13 48.26) (xy 151.13 54.61))
     (stroke (width 0) (type default))
@@
     (stroke (width 0) (type default))
   )
-  (wire (pts (xy 125.73 119.38) (xy 125.73 143.51))
-    (stroke (width 0) (type default))
-  )
   (wire (pts (xy 148.59 101.6) (xy 210.82 101.6))
     (stroke (width 0) (type default))
   )
-  (wire (pts (xy 97.79 127) (xy 104.14 127))
-    (stroke (width 0) (type default))
-  )
   (wire (pts (xy 242.57 80.01) (xy 242.57 87.63))
     (stroke (width 0) (type default))
@@
     (stroke (width 0) (type default))
   )
-  (wire (pts (xy 123.19 99.06) (xy 123.19 106.68))
-    (stroke (width 0) (type default))
-  )
-  (wire (pts (xy 123.19 129.54) (xy 123.19 148.59))
-    (stroke (width 0) (type default))
-  )
   (wire (pts (xy 205.74 156.21) (xy 151.13 156.21))
     (stroke (width 0) (type default))
@@
     (stroke (width 0) (type default))
   )
-  (wire (pts (xy 49.53 156.21) (xy 104.14 156.21))
-    (stroke (width 0) (type default))
-  )
   (wire (pts (xy 246.38 55.88) (xy 246.38 48.26))
     (stroke (width 0) (type default))
@@
     (stroke (width 0) (type default))
   )
-  (wire (pts (xy 128.27 116.84) (xy 97.79 116.84))
-    (stroke (width 0) (type default))
-  )
   (wire (pts (xy 166.37 55.88) (xy 166.37 48.26))
     (stroke (width 0) (type default))
@@
     (stroke (width 0) (type default))
   )
-  (wire (pts (xy 104.14 156.21) (xy 151.13 156.21))
+  (wire (pts (xy 64.77 156.21) (xy 151.13 156.21))
     (stroke (width 0) (type default))
   )
@@
   (wire (pts (xy 232.41 54.61) (xy 232.41 64.77))
     (stroke (width 0) (type default))
-  )
-  (wire (pts (xy 97.79 129.54) (xy 123.19 129.54))
-    (stroke (width 0) (type default))
-  )
-  (symbol (lib_id "Connector:Conn_01x10_Socket") (at 92.71 119.38 180) (unit 1)
-    (in_bom yes) (on_board yes) (dnp no) (fields_autoplaced)
-    (property "Reference" "J7" (at 93.345 101.6 0)
-      (effects (font (size 1.27 1.27)))
-    )
-    (property "Value" "Conn_01x10_Socket" (at 93.345 104.14 0)
-      (effects (font (size 1.27 1.27)))
-    )
-    (property "Footprint" "Connector_PinSocket_2.54mm:PinSocket_2x05_P2.54mm_Vertical" (at 92.71 119.38 0)
-      (effects (font (size 1.27 1.27)) hide)
-    )
-    (property "Datasheet" "~" (at 92.71 119.38 0)
-      (effects (font (size 1.27 1.27)) hide)
-    )
-    (pin "1")
-    (pin "10")
-    (pin "2")
-    (pin "3")
-    (pin "4")
-    (pin "5")
-    (pin "6")
-    (pin "7")
-    (pin "8")
-    (pin "9")
-    (instances
-      (project "PiFencePCB"
-        (path "/59c50c86-add7-4f3c-b7b5-b280f7db1c9d"
-          (reference "J7") (unit 1)
-        )
-      )
-    )
   )
   (symbol (lib_id "New_Library:USB_Power_Breakout") (at 196.85 30.48 0) (unit 1)
@@
         )
       )
+    )
+  )
+  (symbol (lib_id "Interface_Ethernet:ENC28J60x-SP") (at 35.56 166.37 0) (unit 1)
+    (in_bom yes) (on_board yes) (dnp no) (fields_autoplaced)
+    (property "Reference" "U2" (at 40.2941 138.43 0)
+      (effects (font (size 1.27 1.27)) (justify left))
+    )
+    (property "Value" "ENC28J60x-SP" (at 40.2941 140.97 0)
+      (effects (font (size 1.27 1.27)) (justify left))
+    )
+    (property "Footprint" "Package_DIP:DIP-28_W7.62mm" (at 54.61 190.5 0)
+      (effects (font (size 1.27 1.27) italic) hide)
+    )
+    (property "Datasheet" "http://ww1.microchip.com/downloads/en/devicedoc/39662e.pdf" (at 35.56 166.37 0)
+      (effects (font (size 1.27 1.27)) hide)
+    )
+    (pin "11")
+    (pin "5")
+    (pin "9")
+    (pin "13")
+    (pin "3")
+    (pin "1")
+    (pin "18")
+    (pin "12")
+    (pin "4")
+    (pin "14")
+    (pin "7")
+    (pin "19")
+    (pin "10")
+    (pin "21")
+    (pin "27")
+    (pin "22")
+    (pin "25")
+    (pin "20")
+    (pin "24")
+    (pin "23")
+    (pin "2")
+    (pin "26")
+    (pin "28")
+    (pin "16")
+    (pin "17")
+    (pin "6")
+    (pin "15")
+    (pin "8")
+    (instances
+      (project "PiFencePCB"
+        (path "/59c50c86-add7-4f3c-b7b5-b280f7db1c9d"
+          (reference "U2") (unit 1)
+        )
+      )
